Commit message: Added IMU, GPS to Galileo

File: urdf/rover.urdf.xacro (robot description, xacro)
@@ -4,4 +4,5 @@
   <xacro:include filename="rover.gazebo"/>
   <xacro:include filename="rover.trans"/>
+  <link name="camera_link"></link>
   <link name="camera_link_optical">
     <inertial>
@@ -23,4 +24,28 @@
     </collision>
   </link>
+  <link name="imu_link"></link>
+  <link name="gps_link"></link>
+  <link name="lidar_link">
+    <inertial>
+      <origin xyz="0.0 0.0 0.0" rpy="0.0 0.0 0.0"/>
+      <mass value="0.26693"/>
+      <inertia ixx="0.0" ixy="0.0" ixz="0.0" iyy="0.0" iyz="0.0" izz="0.0"/>
+    </inertial>
+    <visual>
+      <origin xyz="0.0 0.0 0.0" rpy="0.0 0.0 0.0"/>
+      <geometry>
+          <cylinder radius="0.04" length="0.03"/>
+      </geometry>
+      <material name="blue">
+        <color rgba="0.0 0.0 1.0 1.0"/>
+      </material>
+    </visual>
+    <collision>
+      <origin xyz="0.0 0.0 0.0" rpy="0.0 0.0 0.0"/>
+      <geometry>
+        <cylinder radius="0.08" length="0.05"/>
+      </geometry>
+    </collision>
+  </link>
   <joint name="camera_joint" type="fixed">
     <origin xyz="0.31 0.0 0.1" rpy="0 0 0"/>
@@ -33,4 +58,18 @@
     <origin xyz="0 0 0" rpy="-${pi/2} 0 ${pi/2}"/>
   </joint>
-  <link name="camera_link"></link>
+  <joint name="lidar_joint" type="fixed">
+    <origin xyz="0.21 0.0 0.165" rpy="0.0 0.0 0.0"/>
+    <parent link="base_link"/>
+    <child link="lidar_link"/>
+  </joint>
+  <joint name="imu_joint" type="fixed">
+    <origin xyz="0.0 0.0 0.165" rpy="0.0 0.0 0.0"/>
+    <parent link="base_link"/>
+    <child link="imu_link"/>
+  </joint>
+  <joint name="gps_joint" type="fixed">
+    <origin xyz="-0.1 0.0 0.165" rpy="0.0 0.0 0.0"/>
+    <parent link="base_link"/>
+    <child link="gps_link"/>
+  </joint>
 </robot>

File: urdf/rover_core.xacro (robot description, xacro)
@@ -40,17 +40,13 @@
         <pose>0.125 0 0 0 0 0</pose>
             <geometry>
-                <box size="0.0001 0.15 0.15"/>
-            </geometry>
-            <material>
-	    <script>
-            	<uri>model://anveshak_logo/scripts</uri>
-            	<uri>model://anveshak_logo/textures</uri>
-            	<name>Logo</name>
-	    </script>
+                <box size="0.0001 0.35 0.35"/>
+            </geometry>
+            <material name="logo">
+	    	<texture filename="package://galileo_description/meshes/anveshak_logo/Anveshak.png"/>
             </material>
-        </visual>
-      </link>
+      </visual>
+    </link>
       <joint name="logo_joint" type="fixed">
-        <origin xyz="0.0 0.0 0.27" rpy="0.0 0.0 0.0"/>
+        <origin xyz="0.0 0.0 0.15" rpy="0.0 ${pi/2} 0.0"/>
         <parent link="base_link"/>
         <child link="anveshak_logo"/>
@@ -81,5 +77,5 @@
         <origin xyz="0 0.24 0.05" rpy="0 0 0"/>
         <axis xyz="0 1 0"/>
-        <limit effort="30" velocity="1.0" lower="-0.1" upper="0.15" />
+        <limit effort="30" velocity="1.0" lower="-0.0" upper="0.15" />
     </joint>
     <link name="right_bogie">
@@ -108,5 +104,5 @@
         <origin xyz="0 -0.24 0.05" rpy="0 0 0"/>
         <axis xyz="0 1 0"/>
-        <limit effort="30" velocity="1.0" lower="-0.1" upper="0.15" />
+        <limit effort="30" velocity="1.0" lower="-0.0" upper="0.15" />
     </joint>
     <link name="left_front_wheel">
