Commit message: Added World and Mapping Plugins

File: urdf/rover_core.xacro (robot description, xacro)
@@ -10,4 +10,10 @@
         <color rgba="1 1 1 1"/>
     </material>
+    <link name="odom"></link>
+    <joint name="odom_joint" type="fixed">
+        <origin xyz="0.0 0.0 0.27" rpy="0.0 0.0 0.0"/>
+        <parent link="odom"/>
+        <child link="base_footprint"/>
+    </joint>
     <link name="base_footprint"></link>
     <joint name="base_joint" type="fixed">
